Commit message: add jazzy branch

File: indy_description/urdf/indy.ros2_control.xacro (robot description, xacro)
@@ -10,9 +10,8 @@
             <hardware>
                 <xacro:if value="${sim_gazebo}">
-                    <plugin>gazebo_ros2_control/GazeboSystem</plugin>
+                    <plugin>gz_ros2_control/GazeboSimSystem</plugin>
                 </xacro:if>
                 <xacro:unless value="${sim_gazebo}">
                     <plugin>fake_components/GenericSystem</plugin>
-                    <!-- <param name="fake_sensor_commands">${fake_sensor_commands}</param> -->
                     <param name="state_following_offset">0.0</param>
                 </xacro:unless>
@@ -21,6 +20,6 @@
                 <joint name="${prefix}${joint_index}">
                     <command_interface name="position">
-                        <param name="min">{-2*pi}</param>
-                        <param name="max">{2*pi}</param>
+                        <param name="min">-6.283185</param>
+                        <param name="max">6.283185</param>
                     </command_interface>
                     <command_interface name="velocity">
@@ -28,13 +27,13 @@
                         <param name="max">3.15</param>
                     </command_interface>
-                    <!-- <state_interface name="position"/> -->
                     <state_interface name="position">
                         <param name="initial_value">${initial_positions[joint_index]}</param>
                     </state_interface>
-                    <!-- <state_interface name="velocity"/> -->
                     <state_interface name="velocity">
                         <param name="initial_value">0.0</param>
                     </state_interface>
-                    <state_interface name="effort"/>
+                    <state_interface name="effort">
+                        <param name="initial_value">0.0</param>
+                    </state_interface>
                 </joint>
             </xacro:macro>

File: indy_description/urdf/indy.urdf.xacro (robot description, xacro)
@@ -38,13 +38,10 @@
     </xacro:indy_robot>
     <xacro:if value="$(arg sim_gazebo)">
-        <gazebo reference="world"> </gazebo>
+        <gazebo reference="world"></gazebo>
         <gazebo>
-            <plugin name="gazebo_ros2_control" filename="libgazebo_ros2_control.so" >
-                <parameters>$(arg simulation_controllers)</parameters>
+            <plugin filename="gz_ros2_control-system" name="gz_ros2_control::GazeboSimROS2ControlPlugin">
+            <parameters>$(arg simulation_controllers)</parameters>
             </plugin>
         </gazebo>
-            <!-- <robot_param>robot_description</robot_param> -->
-            <!-- <robot_param_node>robot_state_publisher</robot_param_node> -->
-            <!-- <parameters>$(find indy_gazebo)/controller/indy_controllers_7dof.yaml</parameters> -->
     </xacro:if>
 </robot>

File: indy_description/urdf/indy_macro.xacro (robot description, xacro)
@@ -107,4 +107,5 @@
                     effort="${sec_limits[joint_index]['max_effort']}"
                     velocity="${sec_limits[joint_index]['max_velocity']}"/>
+                    <!-- acceleration="${sec_limits[joint_index]['max_acceleration']}" -->
             </joint>
         </xacro:macro>
@@ -117,5 +118,5 @@
         <xacro:if value="${indy_type == 'indyrp2' or indy_type == 'indyrp2_v2'}">
             <xacro:define_joint joint_index="joint6" link_1_index="link6" link_2_index="link7"/>
-            <joint name="${prefix}tcp" type="fixed">
+            <joint name="${prefix}joint_tcp" type="fixed">
                 <parent link="${prefix}link7"/>
                 <child link="${prefix}tcp"/>
@@ -124,5 +125,5 @@
         </xacro:if>
         <xacro:unless value="${indy_type == 'indyrp2' or indy_type == 'indyrp2_v2'}">
-            <joint name="${prefix}tcp" type="fixed">
+            <joint name="${prefix}joint_tcp" type="fixed">
                 <parent link="${prefix}link6"/>
                 <child link="${prefix}tcp"/>
