Commit message: add docker, add ICoN3, 7L, Nuri3s, 4s, 20c, Opti5

File: indy_description/urdf/indy_macro.xacro (robot description, xacro)
@@ -23,5 +23,25 @@
         <xacro:define_initialize initial_positions_file="${initial_positions_file}"
             visual_parameters_file="${visual_parameters_file}" indy_type="${indy_type}"/>
-        <xacro:property name="indy_material" value="metal_white"/>
+        <xacro:if value="${ indy_type == 'indy7' or indy_type == 'indy7_v2' or indy_type == 'indyrp2' or
+                            indy_type == 'indyrp2_v2' or indy_type == 'indy12' or indy_type == 'indy12_v2' or
+                            indy_type == 'nuri3s' or indy_type == 'nuri4s' or indy_type == 'nuri7c' or indy_type == 'nuri20c' or indy_type == 'opti5'}">
+            <xacro:property name="material_0" value="indy_white"/>
+            <xacro:property name="material_1" value="indy_white"/>
+            <xacro:property name="material_2" value="indy_white"/>
+            <xacro:property name="material_3" value="indy_white"/>
+            <xacro:property name="material_4" value="indy_white"/>
+            <xacro:property name="material_5" value="indy_white"/>
+            <xacro:property name="material_6" value="indy_white"/>
+            <xacro:property name="material_7" value="indy_white"/>
+        </xacro:if>
+        <xacro:if value="${indy_type == 'icon3' or indy_type == 'icon7l'}">
+            <xacro:property name="material_0" value="icon_grey"/>
+            <xacro:property name="material_1" value="icon_green"/>
+            <xacro:property name="material_2" value="icon_green"/>
+            <xacro:property name="material_3" value="icon_green"/>
+            <xacro:property name="material_4" value="icon_green"/>
+            <xacro:property name="material_5" value="icon_grey"/>
+            <xacro:property name="material_6" value="icon_grey"/>
+        </xacro:if>
         <!-- links -  main serial chain -->
         <xacro:macro name="define_link" params="link_index link_mesh">
@@ -34,5 +54,28 @@
                         <xacro:get_mesh name="${link_mesh}" type="visual"/>
                     </geometry>
-                    <material name="${indy_material}"/>
+                    <xacro:if value="${link_index == 'link0'}">
+                        <material name="${material_0}"/>
+                    </xacro:if>
+                    <xacro:if value="${link_index == 'link1'}">
+                        <material name="${material_1}"/>
+                    </xacro:if>
+                    <xacro:if value="${link_index == 'link2'}">
+                        <material name="${material_2}"/>
+                    </xacro:if>
+                    <xacro:if value="${link_index == 'link3'}">
+                        <material name="${material_3}"/>
+                    </xacro:if>
+                    <xacro:if value="${link_index == 'link4'}">
+                        <material name="${material_4}"/>
+                    </xacro:if>
+                    <xacro:if value="${link_index == 'link5'}">
+                        <material name="${material_5}"/>
+                    </xacro:if>
+                    <xacro:if value="${link_index == 'link6'}">
+                        <material name="${material_6}"/>
+                    </xacro:if>
+                    <xacro:if value="${link_index == 'link7'}">
+                        <material name="${material_7}"/>
+                    </xacro:if>
                 </visual>
                 <collision>
