Commit message: add tcp position to kinematics

File: indy_description/urdf/indy_macro.xacro (robot description, xacro)
@@ -160,15 +160,33 @@
         <xacro:if value="${indy_type == 'indyrp2' or indy_type == 'indyrp2_v2'}">
             <xacro:define_joint joint_index="joint6" link_1_index="link6" link_2_index="link7"/>
+            <xacro:property name="config_kinematics_parameters" value="${xacro.load_yaml(kinematics_parameters_file)}"/>
+            <xacro:property name="sec_kinematics" value="${config_kinematics_parameters['kinematics']}" />
             <joint name="${prefix}tcp" type="fixed">
                 <parent link="${prefix}link7"/>
                 <child link="${prefix}tcp"/>
-                <origin xyz="0 0 0.06" rpy="0 0 0"/>
+                <!-- <origin xyz="0 0 0.06" rpy="0 0 0"/> -->
+                <origin
+                    xyz="${sec_kinematics['tcp']['x']}
+                        ${sec_kinematics['tcp']['y']}
+                        ${sec_kinematics['tcp']['z']}"
+                    rpy="${sec_kinematics['tcp']['roll']}
+                        ${sec_kinematics['tcp']['pitch']}
+                        ${sec_kinematics['tcp']['yaw']}"/>
             </joint>
         </xacro:if>
         <xacro:unless value="${indy_type == 'indyrp2' or indy_type == 'indyrp2_v2'}">
+            <xacro:property name="config_kinematics_parameters" value="${xacro.load_yaml(kinematics_parameters_file)}"/>
+            <xacro:property name="sec_kinematics" value="${config_kinematics_parameters['kinematics']}" />
             <joint name="${prefix}tcp" type="fixed">
                 <parent link="${prefix}link6"/>
                 <child link="${prefix}tcp"/>
-                <origin xyz="0 0 0.06" rpy="0 0 0"/>
+                <!-- <origin xyz="0 0 0.06" rpy="0 0 0"/> -->
+                <origin
+                    xyz="${sec_kinematics['tcp']['x']}
+                        ${sec_kinematics['tcp']['y']}
+                        ${sec_kinematics['tcp']['z']}"
+                    rpy="${sec_kinematics['tcp']['roll']}
+                        ${sec_kinematics['tcp']['pitch']}
+                        ${sec_kinematics['tcp']['yaw']}"/>
             </joint>
         </xacro:unless>

File: indy_description/urdf_files/icon3.urdf (robot description, URDF)
Before this commit: robot indy, 9 links, 8 joints
Links:
- link link0: geometry collision mesh filename=file:///home/user/indy-ros2/install/indy_description/share/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; visual mesh filename=file:///home/user/indy-ros2/install/indy_description/share/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
- link link1: geometry collision mesh filename=file:///home/user/indy-ros2/install/indy_description/share/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; visual mesh filename=file:///home/user/indy-ros2/install/indy_description/share/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
- link link2: geometry collision mesh filename=file:///home/user/indy-ros2/install/indy_description/share/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; visual mesh filename=file:///home/user/indy-ros2/install/indy_description/share/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
- link link3: geometry collision mesh filename=file:///home/user/indy-ros2/install/indy_description/share/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; visual mesh filename=file:///home/user/indy-ros2/install/indy_description/share/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
- link link4: geometry collision mesh filename=file:///home/user/indy-ros2/install/indy_description/share/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; visual mesh filename=file:///home/user/indy-ros2/install/indy_description/share/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
- link link5: geometry collision mesh filename=file:///home/user/indy-ros2/install/indy_description/share/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; visual mesh filename=file:///home/user/indy-ros2/install/indy_description/share/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
- link link6: geometry collision mesh filename=file:///home/user/indy-ros2/install/indy_description/share/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; visual mesh filename=file:///home/user/indy-ros2/install/indy_description/share/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
Joints:
- joint joint5: origin xyz=0.0685                          0.0                          0.0 rpy=0.0                         1.570796327                         0.0 -> xyz=0.0685                          0.0                          0.0 rpy=1.570796327                         0.0                         1.570796327
- joint tcp: origin xyz=0 0 0.06 rpy=0 0 0 -> xyz=0.0                          0.0                          0.0 rpy=0.0                         0.0                         0.0

File: indy_description/urdf_files/icon7l.urdf (robot description, URDF)
Before this commit: robot indy, 9 links, 8 joints
Links:
- link link0: geometry collision mesh filename=file:///home/user/indy-ros2/install/indy_description/share/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; visual mesh filename=file:///home/user/indy-ros2/install/indy_description/share/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
- link link1: geometry collision mesh filename=file:///home/user/indy-ros2/install/indy_description/share/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; visual mesh filename=file:///home/user/indy-ros2/install/indy_description/share/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
- link link2: geometry collision mesh filename=file:///home/user/indy-ros2/install/indy_description/share/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; visual mesh filename=file:///home/user/indy-ros2/install/indy_description/share/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
- link link3: geometry collision mesh filename=file:///home/user/indy-ros2/install/indy_description/share/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; visual mesh filename=file:///home/user/indy-ros2/install/indy_description/share/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
- link link4: geometry collision mesh filename=file:///home/user/indy-ros2/install/indy_description/share/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; visual mesh filename=file:///home/user/indy-ros2/install/indy_description/share/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
- link link5: geometry collision mesh filename=file:///home/user/indy-ros2/install/indy_description/share/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; visual mesh filename=file:///home/user/indy-ros2/install/indy_description/share/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
- link link6: geometry collision mesh filename=file:///home/user/indy-ros2/install/indy_description/share/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; visual mesh filename=file:///home/user/indy-ros2/install/indy_description/share/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
Joints:
- joint joint5: origin xyz=0.0                          0.089                          0.0 rpy=-1.570796327                         0.0                         0.0 -> xyz=0.0                          0.089                          0.0 rpy=1.570796327                         0.0                         3.14159265
- joint tcp: origin xyz=0 0 0.06 rpy=0 0 0 -> xyz=0.0                          0.0                          0.0 rpy=0.0                         0.0                         0.0

File: indy_description/urdf_files/indy12.urdf (robot description, URDF)
Before this commit: robot indy, 9 links, 8 joints
Links:
- link link0: geometry collision mesh filename=file:///home/user/indy-ros2/install/indy_description/share/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; visual mesh filename=file:///home/user/indy-ros2/install/indy_description/share/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
- link link1: geometry collision mesh filename=file:///home/user/indy-ros2/install/indy_description/share/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; visual mesh filename=file:///home/user/indy-ros2/install/indy_description/share/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
- link link2: geometry collision mesh filename=file:///home/user/indy-ros2/install/indy_description/share/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; visual mesh filename=file:///home/user/indy-ros2/install/indy_description/share/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
- link link3: geometry collision mesh filename=file:///home/user/indy-ros2/install/indy_description/share/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; visual mesh filename=file:///home/user/indy-ros2/install/indy_description/share/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
- link link4: geometry collision mesh filename=file:///home/user/indy-ros2/install/indy_description/share/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; visual mesh filename=file:///home/user/indy-ros2/install/indy_description/share/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
- link link5: geometry collision mesh filename=file:///home/user/indy-ros2/install/indy_description/share/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; visual mesh filename=file:///home/user/indy-ros2/install/indy_description/share/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
- link link6: geometry collision mesh filename=file:///home/user/indy-ros2/install/indy_description/share/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; visual mesh filename=file:///home/user/indy-ros2/install/indy_description/share/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
Joints:
- joint tcp: origin xyz=0 0 0.06 rpy=0 0 0 -> xyz=0.0                          0.0                          0.06 rpy=0.0                         0.0                         0.0

File: indy_description/urdf_files/indy12_v2.urdf (robot description, URDF)
Before this commit: robot indy, 9 links, 8 joints
Links:
- link link0: geometry collision mesh filename=file:///home/user/indy-ros2/install/indy_description/share/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; visual mesh filename=file:///home/user/indy-ros2/install/indy_description/share/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
- link link1: geometry collision mesh filename=file:///home/user/indy-ros2/install/indy_description/share/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; visual mesh filename=file:///home/user/indy-ros2/install/indy_description/share/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
- link link2: geometry collision mesh filename=file:///home/user/indy-ros2/install/indy_description/share/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; visual mesh filename=file:///home/user/indy-ros2/install/indy_description/share/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
- link link3: geometry collision mesh filename=file:///home/user/indy-ros2/install/indy_description/share/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; visual mesh filename=file:///home/user/indy-ros2/install/indy_description/share/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
- link link4: geometry collision mesh filename=file:///home/user/indy-ros2/install/indy_description/share/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; visual mesh filename=file:///home/user/indy-ros2/install/indy_description/share/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
- link link5: geometry collision mesh filename=file:///home/user/indy-ros2/install/indy_description/share/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; visual mesh filename=file:///home/user/indy-ros2/install/indy_description/share/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
- link link6: geometry collision mesh filename=file:///home/user/indy-ros2/install/indy_description/share/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; visual mesh filename=file:///home/user/indy-ros2/install/indy_description/share/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
Joints:
- joint tcp: origin xyz=0 0 0.06 rpy=0 0 0 -> xyz=0.0                          0.0                          0.09 rpy=0.0                         0.0                         0.0

File: indy_description/urdf_files/indy7.urdf (robot description, URDF)
Before this commit: robot indy, 9 links, 8 joints
Links:
- link link0: geometry collision mesh filename=file:///home/user/indy-ros2/install/indy_description/share/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; visual mesh filename=file:///home/user/indy-ros2/install/indy_description/share/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
- link link1: geometry collision mesh filename=file:///home/user/indy-ros2/install/indy_description/share/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; visual mesh filename=file:///home/user/indy-ros2/install/indy_description/share/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
- link link2: geometry collision mesh filename=file:///home/user/indy-ros2/install/indy_description/share/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; visual mesh filename=file:///home/user/indy-ros2/install/indy_description/share/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
- link link3: geometry collision mesh filename=file:///home/user/indy-ros2/install/indy_description/share/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; visual mesh filename=file:///home/user/indy-ros2/install/indy_description/share/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
- link link4: geometry collision mesh filename=file:///home/user/indy-ros2/install/indy_description/share/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; visual mesh filename=file:///home/user/indy-ros2/install/indy_description/share/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
- link link5: geometry collision mesh filename=file:///home/user/indy-ros2/install/indy_description/share/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; visual mesh filename=file:///home/user/indy-ros2/install/indy_description/share/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
- link link6: geometry collision mesh filename=file:///home/user/indy-ros2/install/indy_description/share/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; visual mesh filename=file:///home/user/indy-ros2/install/indy_description/share/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
Joints:
- joint tcp: origin xyz=0 0 0.06 rpy=0 0 0 -> xyz=0.0                          0.0                          0.06 rpy=0.0                         0.0                         0.0

File: indy_description/urdf_files/indy7_eye.urdf (robot description, URDF)
Before this commit: robot indy, 9 links, 8 joints
Links:
- link link0: geometry collision mesh filename=file:///home/user/indy-ros2/install/indy_description/share/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; visual mesh filename=file:///home/user/indy-ros2/install/indy_description/share/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
- link link1: geometry collision mesh filename=file:///home/user/indy-ros2/install/indy_description/share/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; visual mesh filename=file:///home/user/indy-ros2/install/indy_description/share/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
- link link2: geometry collision mesh filename=file:///home/user/indy-ros2/install/indy_description/share/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; visual mesh filename=file:///home/user/indy-ros2/install/indy_description/share/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
- link link3: geometry collision mesh filename=file:///home/user/indy-ros2/install/indy_description/share/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; visual mesh filename=file:///home/user/indy-ros2/install/indy_description/share/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
- link link4: geometry collision mesh filename=file:///home/user/indy-ros2/install/indy_description/share/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; visual mesh filename=file:///home/user/indy-ros2/install/indy_description/share/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
- link link5: geometry collision mesh filename=file:///home/user/indy-ros2/install/indy_description/share/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; visual mesh filename=file:///home/user/indy-ros2/install/indy_description/share/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
- link link6: geometry collision mesh filename=file:///home/user/indy-ros2/install/indy_description/share/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; visual mesh filename=file:///home/user/indy-ros2/install/indy_description/share/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
Joints:
- joint tcp: origin xyz=0 0 0.06 rpy=0 0 0 -> xyz=0.0                          0.0                          0.06 rpy=0.0                         0.0                         0.0

File: indy_description/urdf_files/indy7_v2.urdf (robot description, URDF)
Before this commit: robot indy, 9 links, 8 joints
Links:
- link link0: geometry collision mesh filename=file:///home/user/indy-ros2/install/indy_description/share/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; visual mesh filename=file:///home/user/indy-ros2/install/indy_description/share/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
- link link1: geometry collision mesh filename=file:///home/user/indy-ros2/install/indy_description/share/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; visual mesh filename=file:///home/user/indy-ros2/install/indy_description/share/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
- link link2: geometry collision mesh filename=file:///home/user/indy-ros2/install/indy_description/share/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; visual mesh filename=file:///home/user/indy-ros2/install/indy_description/share/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
- link link3: geometry collision mesh filename=file:///home/user/indy-ros2/install/indy_description/share/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; visual mesh filename=file:///home/user/indy-ros2/install/indy_description/share/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
- link link4: geometry collision mesh filename=file:///home/user/indy-ros2/install/indy_description/share/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; visual mesh filename=file:///home/user/indy-ros2/install/indy_description/share/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
- link link5: geometry collision mesh filename=file:///home/user/indy-ros2/install/indy_description/share/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; visual mesh filename=file:///home/user/indy-ros2/install/indy_description/share/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
- link link6: geometry collision mesh filename=file:///home/user/indy-ros2/install/indy_description/share/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; visual mesh filename=file:///home/user/indy-ros2/install/indy_description/share/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
Joints:
- joint tcp: origin xyz=0 0 0.06 rpy=0 0 0 -> xyz=0.0                          0.0                          0.06 rpy=0.0                         0.0                         0.0

File: indy_description/urdf_files/indyrp2.urdf (robot description, URDF)
Before this commit: robot indy, 10 links, 9 joints
Links:
- link link0: geometry collision mesh filename=file:///home/user/indy-ros2/install/indy_description/share/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; visual mesh filename=file:///home/user/indy-ros2/install/indy_description/share/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
- link link1: geometry collision mesh filename=file:///home/user/indy-ros2/install/indy_description/share/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; visual mesh filename=file:///home/user/indy-ros2/install/indy_description/share/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
- link link2: geometry collision mesh filename=file:///home/user/indy-ros2/install/indy_description/share/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; visual mesh filename=file:///home/user/indy-ros2/install/indy_description/share/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
- link link3: geometry collision mesh filename=file:///home/user/indy-ros2/install/indy_description/share/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; visual mesh filename=file:///home/user/indy-ros2/install/indy_description/share/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
- link link4: geometry collision mesh filename=file:///home/user/indy-ros2/install/indy_description/share/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; visual mesh filename=file:///home/user/indy-ros2/install/indy_description/share/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
- link link5: geometry collision mesh filename=file:///home/user/indy-ros2/install/indy_description/share/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; visual mesh filename=file:///home/user/indy-ros2/install/indy_description/share/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
- link link6: geometry collision mesh filename=file:///home/user/indy-ros2/install/indy_description/share/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; visual mesh filename=file:///home/user/indy-ros2/install/indy_description/share/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
- link link7: geometry collision mesh filename=file:///home/user/indy-ros2/install/indy_description/share/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; visual mesh filename=file:///home/user/indy-ros2/install/indy_description/share/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
Joints:
- joint tcp: origin xyz=0 0 0.06 rpy=0 0 0 -> xyz=0.0                          0.0                          0.06 rpy=0.0                         0.0                         0.0

File: indy_description/urdf_files/indyrp2_eye.urdf (robot description, URDF)
Before this commit: robot indy, 10 links, 9 joints
Links:
- link link0: geometry collision mesh filename=file:///home/user/indy-ros2/install/indy_description/share/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; visual mesh filename=file:///home/user/indy-ros2/install/indy_description/share/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
- link link1: geometry collision mesh filename=file:///home/user/indy-ros2/install/indy_description/share/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; visual mesh filename=file:///home/user/indy-ros2/install/indy_description/share/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
- link link2: geometry collision mesh filename=file:///home/user/indy-ros2/install/indy_description/share/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; visual mesh filename=file:///home/user/indy-ros2/install/indy_description/share/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
- link link3: geometry collision mesh filename=file:///home/user/indy-ros2/install/indy_description/share/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; visual mesh filename=file:///home/user/indy-ros2/install/indy_description/share/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
- link link4: geometry collision mesh filename=file:///home/user/indy-ros2/install/indy_description/share/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; visual mesh filename=file:///home/user/indy-ros2/install/indy_description/share/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
- link link5: geometry collision mesh filename=file:///home/user/indy-ros2/install/indy_description/share/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; visual mesh filename=file:///home/user/indy-ros2/install/indy_description/share/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
- link link6: geometry collision mesh filename=file:///home/user/indy-ros2/install/indy_description/share/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; visual mesh filename=file:///home/user/indy-ros2/install/indy_description/share/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
- link link7: geometry collision mesh filename=file:///home/user/indy-ros2/install/indy_description/share/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; visual mesh filename=file:///home/user/indy-ros2/install/indy_description/share/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
Joints:
- joint tcp: origin xyz=0 0 0.06 rpy=0 0 0 -> xyz=0.0                          0.0                          0.06 rpy=0.0                         0.0                         0.0

File: indy_description/urdf_files/indyrp2_v2.urdf (robot description, URDF)
Before this commit: robot indy, 10 links, 9 joints
Links:
- link link0: geometry collision mesh filename=file:///home/user/indy-ros2/install/indy_description/share/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; visual mesh filename=file:///home/user/indy-ros2/install/indy_description/share/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
- link link1: geometry collision mesh filename=file:///home/user/indy-ros2/install/indy_description/share/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; visual mesh filename=file:///home/user/indy-ros2/install/indy_description/share/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
- link link2: geometry collision mesh filename=file:///home/user/indy-ros2/install/indy_description/share/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; visual mesh filename=file:///home/user/indy-ros2/install/indy_description/share/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
- link link3: geometry collision mesh filename=file:///home/user/indy-ros2/install/indy_description/share/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; visual mesh filename=file:///home/user/indy-ros2/install/indy_description/share/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
- link link4: geometry collision mesh filename=file:///home/user/indy-ros2/install/indy_description/share/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; visual mesh filename=file:///home/user/indy-ros2/install/indy_description/share/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
- link link5: geometry collision mesh filename=file:///home/user/indy-ros2/install/indy_description/share/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; visual mesh filename=file:///home/user/indy-ros2/install/indy_description/share/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
- link link6: geometry collision mesh filename=file:///home/user/indy-ros2/install/indy_description/share/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; visual mesh filename=file:///home/user/indy-ros2/install/indy_description/share/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
- link link7: geometry collision mesh filename=file:///home/user/indy-ros2/install/indy_description/share/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; visual mesh filename=file:///home/user/indy-ros2/install/indy_description/share/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
Joints:
- joint tcp: origin xyz=0 0 0.06 rpy=0 0 0 -> xyz=0.0                          0.0                          0.06 rpy=0.0                         0.0                         0.0

File: indy_description/urdf_files/nuri20c.urdf (robot description, URDF)
Before this commit: robot indy, 9 links, 8 joints
Links:
- link link0: mass 0.858186768 -> 10.512390866; geometry collision mesh filename=file:///home/user/indy-ros2/install/indy_description/share/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; visual mesh filename=file:///home/user/indy-ros2/install/indy_description/share/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
- link link1: mass 2.520440484 -> 18.195720206; geometry collision mesh filename=file:///home/user/indy-ros2/install/indy_description/share/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; visual mesh filename=file:///home/user/indy-ros2/install/indy_description/share/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
- link link2: mass 3.1785267 -> 22.845886455; geometry collision mesh filename=file:///home/user/indy-ros2/install/indy_description/share/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; visual mesh filename=file:///home/user/indy-ros2/install/indy_description/share/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
- link link3: mass 1.601379441 -> 7.83830585; geometry collision mesh filename=file:///home/user/indy-ros2/install/indy_description/share/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; visual mesh filename=file:///home/user/indy-ros2/install/indy_description/share/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
- link link4: mass 1.882223023 -> 6.943393986; geometry collision mesh filename=file:///home/user/indy-ros2/install/indy_description/share/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; visual mesh filename=file:///home/user/indy-ros2/install/indy_description/share/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
- link link5: mass 1.507185922 -> 3.229294314; geometry collision mesh filename=file:///home/user/indy-ros2/install/indy_description/share/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; visual mesh filename=file:///home/user/indy-ros2/install/indy_description/share/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
- link link6: mass 0.634034296 -> 1.586348204; geometry collision mesh filename=file:///home/user/indy-ros2/install/indy_description/share/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; visual mesh filename=file:///home/user/indy-ros2/install/indy_description/share/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
Joints:
- joint tcp: origin xyz=0 0 0.06 rpy=0 0 0 -> xyz=0.0                          0.0                          0.04 rpy=0.0                         0.0                         0.0
