Commit message: add tcp position to kinematics

File: indy_description/urdf_files/nuri3s.urdf (robot description, URDF)
Before this commit: robot indy, 9 links, 8 joints
Links:
- link link0: geometry collision mesh filename=file:///home/user/indy-ros2/install/indy_description/share/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; visual mesh filename=file:///home/user/indy-ros2/install/indy_description/share/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
- link link1: geometry collision mesh filename=file:///home/user/indy-ros2/install/indy_description/share/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; visual mesh filename=file:///home/user/indy-ros2/install/indy_description/share/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
- link link2: geometry collision mesh filename=file:///home/user/indy-ros2/install/indy_description/share/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; visual mesh filename=file:///home/user/indy-ros2/install/indy_description/share/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
- link link3: geometry collision mesh filename=file:///home/user/indy-ros2/install/indy_description/share/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; visual mesh filename=file:///home/user/indy-ros2/install/indy_description/share/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
- link link4: geometry collision mesh filename=file:///home/user/indy-ros2/install/indy_description/share/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; visual mesh filename=file:///home/user/indy-ros2/install/indy_description/share/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
- link link5: geometry collision mesh filename=file:///home/user/indy-ros2/install/indy_description/share/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; visual mesh filename=file:///home/user/indy-ros2/install/indy_description/share/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
- link link6: geometry collision mesh filename=file:///home/user/indy-ros2/install/indy_description/share/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; visual mesh filename=file:///home/user/indy-ros2/install/indy_description/share/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
Joints:
- joint tcp: origin xyz=0 0 0.06 rpy=0 0 0 -> xyz=0.0                          0.0                          0.0285 rpy=0.0                         0.0                         0.0

File: indy_description/urdf_files/nuri4s.urdf (robot description, URDF)
Before this commit: robot indy, 9 links, 8 joints
Links:
- link link0: mass 0.858186768 -> 2.861045494; geometry collision mesh filename=file:///home/user/indy-ros2/install/indy_description/share/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; visual mesh filename=file:///home/user/indy-ros2/install/indy_description/share/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
- link link1: mass 2.520440484 -> 3.167175036; geometry collision mesh filename=file:///home/user/indy-ros2/install/indy_description/share/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; visual mesh filename=file:///home/user/indy-ros2/install/indy_description/share/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
- link link2: mass 3.1785267 -> 4.29096783; geometry collision mesh filename=file:///home/user/indy-ros2/install/indy_description/share/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; visual mesh filename=file:///home/user/indy-ros2/install/indy_description/share/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
- link link3: mass 1.601379441 -> 2.018198648; geometry collision mesh filename=file:///home/user/indy-ros2/install/indy_description/share/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; visual mesh filename=file:///home/user/indy-ros2/install/indy_description/share/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
- link link4: geometry collision mesh filename=file:///home/user/indy-ros2/install/indy_description/share/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; visual mesh filename=file:///home/user/indy-ros2/install/indy_description/share/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
- link link5: geometry collision mesh filename=file:///home/user/indy-ros2/install/indy_description/share/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; visual mesh filename=file:///home/user/indy-ros2/install/indy_description/share/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
- link link6: geometry collision mesh filename=file:///home/user/indy-ros2/install/indy_description/share/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; visual mesh filename=file:///home/user/indy-ros2/install/indy_description/share/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
Joints:
- joint tcp: origin xyz=0 0 0.06 rpy=0 0 0 -> xyz=0.0                          0.0                          0.0285 rpy=0.0                         0.0                         0.0

File: indy_description/urdf_files/nuri7c.urdf (robot description, URDF)
Before this commit: robot indy, 9 links, 8 joints
Links:
- link link0: mass 0.858186768 -> 4.23; geometry collision mesh filename=file:///home/user/indy-ros2/install/indy_description/share/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; visual mesh filename=file:///home/user/indy-ros2/install/indy_description/share/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
- link link1: mass 2.520440484 -> 5.489055681; geometry collision mesh filename=file:///home/user/indy-ros2/install/indy_description/share/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; visual mesh filename=file:///home/user/indy-ros2/install/indy_description/share/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
- link link2: mass 3.1785267 -> 7.28078719; geometry collision mesh filename=file:///home/user/indy-ros2/install/indy_description/share/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; visual mesh filename=file:///home/user/indy-ros2/install/indy_description/share/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
- link link3: mass 1.601379441 -> 2.871921442; geometry collision mesh filename=file:///home/user/indy-ros2/install/indy_description/share/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; visual mesh filename=file:///home/user/indy-ros2/install/indy_description/share/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
- link link4: mass 1.882223023 -> 2.822752725; geometry collision mesh filename=file:///home/user/indy-ros2/install/indy_description/share/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; visual mesh filename=file:///home/user/indy-ros2/install/indy_description/share/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
- link link5: mass 1.507185922 -> 2.340109457; geometry collision mesh filename=file:///home/user/indy-ros2/install/indy_description/share/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; visual mesh filename=file:///home/user/indy-ros2/install/indy_description/share/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
- link link6: mass 0.634034296 -> 1.141750934; geometry collision mesh filename=file:///home/user/indy-ros2/install/indy_description/share/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; visual mesh filename=file:///home/user/indy-ros2/install/indy_description/share/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
Joints:
- joint tcp: origin xyz=0 0 0.06 rpy=0 0 0 -> xyz=0.0                          0.0                          0.054 rpy=0.0                         0.0                         0.0

File: indy_description/urdf_files/opti5.urdf (robot description, URDF)
Before this commit: robot indy, 9 links, 8 joints
Links:
- link link0: geometry collision mesh filename=file:///home/user/indy-ros2/install/indy_description/share/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; visual mesh filename=file:///home/user/indy-ros2/install/indy_description/share/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
- link link1: geometry collision mesh filename=file:///home/user/indy-ros2/install/indy_description/share/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; visual mesh filename=file:///home/user/indy-ros2/install/indy_description/share/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
- link link2: geometry collision mesh filename=file:///home/user/indy-ros2/install/indy_description/share/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; visual mesh filename=file:///home/user/indy-ros2/install/indy_description/share/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
- link link3: geometry collision mesh filename=file:///home/user/indy-ros2/install/indy_description/share/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; visual mesh filename=file:///home/user/indy-ros2/install/indy_description/share/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
- link link4: geometry collision mesh filename=file:///home/user/indy-ros2/install/indy_description/share/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; visual mesh filename=file:///home/user/indy-ros2/install/indy_description/share/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
- link link5: geometry collision mesh filename=file:///home/user/indy-ros2/install/indy_description/share/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; visual mesh filename=file:///home/user/indy-ros2/install/indy_description/share/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
- link link6: geometry collision mesh filename=file:///home/user/indy-ros2/install/indy_description/share/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; visual mesh filename=file:///home/user/indy-ros2/install/indy_description/share/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
Joints:
- joint tcp: origin xyz=0 0 0.06 rpy=0 0 0 -> xyz=0.0                          0.0                          0.0605 rpy=0.0                         0.0                         0.0
