Commit message: foxy->humble

File: indy_description/urdf/indy_common.xacro (robot description, xacro)
@@ -14,5 +14,5 @@
     </xacro:macro>
     <xacro:macro name="define_initialize" params="visual_parameters_file">
-        <xacro:property name="config_visual_parameters" value="${load_yaml(visual_parameters_file)}"/>
+        <xacro:property name="config_visual_parameters" value="${xacro.load_yaml(visual_parameters_file)}"/>
         <xacro:property name="sec_mesh_files" value="${config_visual_parameters['mesh_files']}" scope="parent"/>
     </xacro:macro>

File: indy_description/urdf/indy_macro.xacro (robot description, xacro)
@@ -25,5 +25,5 @@
         <xacro:macro name="define_link" params="link_index link_mesh">
             <link name="${prefix}${link_index}">
-                <xacro:property name="config_physical_parameters" value="${load_yaml(physical_parameters_file)}"/>
+                <xacro:property name="config_physical_parameters" value="${xacro.load_yaml(physical_parameters_file)}"/>
                 <xacro:property name="sec_inertia_parameters" value="${config_physical_parameters['inertia_parameters']}" />
                 <visual>
@@ -85,6 +85,6 @@
         </joint>
         <xacro:macro name="define_joint" params="joint_index link_1_index link_2_index" >
-            <xacro:property name="config_joint_limit_parameters" value="${load_yaml(joint_limits_parameters_file)}"/>
-            <xacro:property name="config_kinematics_parameters" value="${load_yaml(kinematics_parameters_file)}"/>
+            <xacro:property name="config_joint_limit_parameters" value="${xacro.load_yaml(joint_limits_parameters_file)}"/>
+            <xacro:property name="config_kinematics_parameters" value="${xacro.load_yaml(kinematics_parameters_file)}"/>
             <xacro:property name="sec_kinematics" value="${config_kinematics_parameters['kinematics']}" />
             <xacro:property name="sec_limits" value="${config_joint_limit_parameters['joint_limits']}"/>
