Commit message: add urdf generator, add model for Nuri7c

File: indy_description/urdf_files/nuri20c.urdf (robot description, URDF)
Before this commit: robot indy, 9 links, 8 joints
Links:
- link link0: mass 13.983 -> 0.858186768
- link link1: mass 10.239 -> 2.520440484
- link link2: mass 12.857 -> 3.1785267
- link link3: mass 7.462 -> 1.601379441
- link link4: mass 4.38 -> 1.882223023
- link link5: mass 1.656 -> 1.507185922
- link link6: mass 0.272 -> 0.634034296
Joints:
- joint joint0: limit lower=-2.9670597283903604 upper=2.9670597283903604 effort=431.97 velocity=6.632251157578453 -> lower=-6.283185307179586 upper=6.283185307179586 effort=431.97 velocity=3.141592653589793; origin xyz=0.0                          0.0                          0.19825 rpy=0.0                         0.0                         0.0 -> xyz=0.0                          0.0                          0.079 rpy=0.0                         0.0                         0.0
- joint joint1: limit lower=-1.7453292519943295 upper=2.356194490192345 effort=431.97 velocity=5.585053606381854 -> lower=-2.705260340591211 upper=2.443460952792061 effort=431.97 velocity=3.141592653589793; origin xyz=0.025                          0.0                          0.202 rpy=-1.570796327                         0.0                         0.0 -> xyz=0.0                          -0.12                          0.288 rpy=1.570796327                         0.0                         0.0
- joint joint2: limit lower=-2.0943951023931953 upper=2.722713633111154 effort=197.23 velocity=6.806784082777885 -> lower=-3.0543261909900767 upper=2.356194490192345 effort=197.23 velocity=3.141592653589793; origin xyz=0.0                          -0.463                          0.0 rpy=0.0                         0.0                         0.0 -> xyz=0.0                          0.9                          0.0 rpy=0.0                         0.0                         0.0
- joint joint3: limit lower=-3.490658503988659 upper=3.490658503988659 effort=79.79 velocity=8.552113334772216 -> lower=-6.283185307179586 upper=6.283185307179586 effort=79.79 velocity=3.141592653589793; origin xyz=-0.035                          -0.182                          0.0 rpy=1.570796327                         1.570796327                         0.0 -> xyz=0.0                          0.22                          -0.12 rpy=-1.570796327                         0.0                         0.0
- joint joint4: limit lower=-2.356194490192345 upper=2.356194490192345 effort=79.79 velocity=9.861110273767961 -> lower=-6.283185307179586 upper=6.283185307179586 effort=79.79 velocity=3.141592653589793; origin xyz=0.0                          0.0                          0.25 rpy=1.570796327                         0.0                         -1.570796327 -> xyz=0.0                          0.11                          0.53 rpy=1.570796327                         0.0                         0.0
- joint joint5: limit lower=-6.283185307179586 upper=6.283185307179586 effort=79.79 velocity=14.224433403753785 -> lower=-6.283185307179586 upper=6.283185307179586 effort=79.79 velocity=3.141592653589793; origin xyz=0.0                          0.089                          0.0 rpy=-1.570796327                         0.0                         0.0 -> xyz=0.0                          0.1                          -0.06 rpy=-1.570796327                         0.0                         0.0

File: indy_description/urdf_files/nuri3s.urdf (robot description, URDF)
Before this commit: robot indy, 9 links, 8 joints
Links:
- link link0: mass 13.983 -> 0.858186768
- link link1: mass 10.239 -> 2.520440484
- link link2: mass 12.857 -> 3.1785267
- link link3: mass 7.462 -> 1.601379441
- link link4: mass 4.38 -> 1.882223023
- link link5: mass 1.656 -> 1.507185922
- link link6: mass 0.272 -> 0.634034296
Joints:
- joint joint0: limit lower=-2.9670597283903604 upper=2.9670597283903604 effort=431.97 velocity=6.632251157578453 -> lower=-6.283185307179586 upper=6.283185307179586 effort=431.97 velocity=3.141592653589793; origin xyz=0.0                          0.0                          0.19825 rpy=0.0                         0.0                         0.0 -> xyz=0.0                          0.0                          0.09 rpy=0.0                         0.0                         0.0
- joint joint1: limit lower=-1.7453292519943295 upper=2.356194490192345 effort=431.97 velocity=5.585053606381854 -> lower=-2.705260340591211 upper=2.443460952792061 effort=431.97 velocity=3.141592653589793; origin xyz=0.025                          0.0                          0.202 rpy=-1.570796327                         0.0                         0.0 -> xyz=0.0                          -0.04                          0.223 rpy=1.570796327                         0.0                         0.0
- joint joint2: limit lower=-2.0943951023931953 upper=2.722713633111154 effort=197.23 velocity=6.806784082777885 -> lower=-3.0543261909900767 upper=2.356194490192345 effort=197.23 velocity=3.141592653589793; origin xyz=0.0                          -0.463                          0.0 rpy=0.0                         0.0                         0.0 -> xyz=0.05023                          0.2900135                          0.0 rpy=0.0                         0.0                         0.0
- joint joint3: limit lower=-3.490658503988659 upper=3.490658503988659 effort=79.79 velocity=8.552113334772216 -> lower=-6.283185307179586 upper=6.283185307179586 effort=79.79 velocity=3.141592653589793; origin xyz=-0.035                          -0.182                          0.0 rpy=1.570796327                         1.570796327                         0.0 -> xyz=-0.05                          0.085                          -0.04 rpy=-1.570796327                         0.0                         0.0
- joint joint4: limit lower=-2.356194490192345 upper=2.356194490192345 effort=79.79 velocity=9.861110273767961 -> lower=-6.283185307179586 upper=6.283185307179586 effort=79.79 velocity=3.141592653589793; origin xyz=0.0                          0.0                          0.25 rpy=1.570796327                         0.0                         -1.570796327 -> xyz=0.0                          0.07                          0.2050424 rpy=1.570796327                         0.0                         0.0
- joint joint5: limit lower=-6.283185307179586 upper=6.283185307179586 effort=79.79 velocity=14.224433403753785 -> lower=-6.283185307179586 upper=6.283185307179586 effort=79.79 velocity=3.141592653589793; origin xyz=0.0                          0.089                          0.0 rpy=-1.570796327                         0.0                         0.0 -> xyz=0.0                          0.075                          -0.066 rpy=-1.570796327                         0.0                         0.0

File: indy_description/urdf_files/nuri4s.urdf (robot description, URDF)
Before this commit: robot indy, 9 links, 8 joints
Links:
- link link0: mass 13.983 -> 0.858186768
- link link1: mass 10.239 -> 2.520440484
- link link2: mass 12.857 -> 3.1785267
- link link3: mass 7.462 -> 1.601379441
- link link4: mass 4.38 -> 1.882223023
- link link5: mass 1.656 -> 1.507185922
- link link6: mass 0.272 -> 0.634034296
Joints:
- joint joint0: limit lower=-2.9670597283903604 upper=2.9670597283903604 effort=431.97 velocity=6.632251157578453 -> lower=-6.283185307179586 upper=6.283185307179586 effort=431.97 velocity=3.141592653589793; origin xyz=0.0                          0.0                          0.19825 rpy=0.0                         0.0                         0.0 -> xyz=0.0                          0.0                          0.09 rpy=0.0                         0.0                         0.0
- joint joint1: limit lower=-1.7453292519943295 upper=2.356194490192345 effort=431.97 velocity=5.585053606381854 -> lower=-2.705260340591211 upper=2.443460952792061 effort=431.97 velocity=3.141592653589793; origin xyz=0.025                          0.0                          0.202 rpy=-1.570796327                         0.0                         0.0 -> xyz=0.0                          -0.04                          0.238 rpy=1.570796327                         0.0                         0.0
- joint joint2: limit lower=-2.0943951023931953 upper=2.722713633111154 effort=197.23 velocity=6.806784082777885 -> lower=-3.0543261909900767 upper=2.356194490192345 effort=197.23 velocity=3.141592653589793; origin xyz=0.0                          -0.463                          0.0 rpy=0.0                         0.0                         0.0 -> xyz=0.05                          0.4                          0.0 rpy=0.0                         0.0                         0.0
- joint joint3: limit lower=-3.490658503988659 upper=3.490658503988659 effort=79.79 velocity=8.552113334772216 -> lower=-6.283185307179586 upper=6.283185307179586 effort=79.79 velocity=3.141592653589793; origin xyz=-0.035                          -0.182                          0.0 rpy=1.570796327                         1.570796327                         0.0 -> xyz=-0.05                          0.195                          -0.04 rpy=-1.570796327                         0.0                         0.0
- joint joint4: limit lower=-2.356194490192345 upper=2.356194490192345 effort=79.79 velocity=9.861110273767961 -> lower=-6.283185307179586 upper=6.283185307179586 effort=79.79 velocity=3.141592653589793; origin xyz=0.0                          0.0                          0.25 rpy=1.570796327                         0.0                         -1.570796327 -> xyz=0.0                          0.07                          0.2050424 rpy=1.570796327                         0.0                         0.0
- joint joint5: limit lower=-6.283185307179586 upper=6.283185307179586 effort=79.79 velocity=14.224433403753785 -> lower=-6.283185307179586 upper=6.283185307179586 effort=79.79 velocity=3.141592653589793; origin xyz=0.0                          0.089                          0.0 rpy=-1.570796327                         0.0                         0.0 -> xyz=0.0                          0.075                          -0.066 rpy=-1.570796327                         0.0                         0.0

File: indy_description/urdf_files/nuri7c.urdf (robot description, URDF)
Before this commit: robot indy, 9 links, 8 joints
Links:
- link link0: mass 13.983 -> 0.858186768
- link link1: mass 10.239 -> 2.520440484
- link link2: mass 12.857 -> 3.1785267
- link link3: mass 7.462 -> 1.601379441
- link link4: mass 4.38 -> 1.882223023
- link link5: mass 1.656 -> 1.507185922
- link link6: mass 0.272 -> 0.634034296
Joints:
- joint joint0: limit lower=-2.9670597283903604 upper=2.9670597283903604 effort=431.97 velocity=6.632251157578453 -> lower=-6.283185307179586 upper=6.283185307179586 effort=431.97 velocity=3.141592653589793; origin xyz=0.0                          0.0                          0.19825 rpy=0.0                         0.0                         0.0 -> xyz=0.0                          0.0                          0.0705 rpy=0.0                         0.0                         0.0
- joint joint1: limit lower=-1.7453292519943295 upper=2.356194490192345 effort=431.97 velocity=5.585053606381854 -> lower=-2.705260340591211 upper=2.443460952792061 effort=431.97 velocity=3.141592653589793; origin xyz=0.025                          0.0                          0.202 rpy=-1.570796327                         0.0                         0.0 -> xyz=0.0                          -0.0915                          0.171 rpy=1.570796327                         0.0                         0.0
- joint joint2: limit lower=-2.0943951023931953 upper=2.722713633111154 effort=197.23 velocity=6.806784082777885 -> lower=-3.0543261909900767 upper=2.356194490192345 effort=197.23 velocity=3.141592653589793; origin xyz=0.0                          -0.463                          0.0 rpy=0.0                         0.0                         0.0 -> xyz=0.0                          0.49                          0.0 rpy=0.0                         0.0                         0.0
- joint joint3: limit lower=-3.490658503988659 upper=3.490658503988659 effort=79.79 velocity=8.552113334772216 -> lower=-6.283185307179586 upper=6.283185307179586 effort=79.79 velocity=3.141592653589793; origin xyz=-0.035                          -0.182                          0.0 rpy=1.570796327                         1.570796327                         0.0 -> xyz=0.0                          0.1475                          -0.0915 rpy=-1.570796327                         0.0                         0.0
- joint joint4: limit lower=-2.356194490192345 upper=2.356194490192345 effort=79.79 velocity=9.861110273767961 -> lower=-6.283185307179586 upper=6.283185307179586 effort=79.79 velocity=3.141592653589793; origin xyz=0.0                          0.0                          0.25 rpy=1.570796327                         0.0                         -1.570796327 -> xyz=0.0                          0.0737                          0.2125 rpy=1.570796327                         0.0                         0.0
- joint joint5: limit lower=-6.283185307179586 upper=6.283185307179586 effort=79.79 velocity=14.224433403753785 -> lower=-6.283185307179586 upper=6.283185307179586 effort=79.79 velocity=3.141592653589793; origin xyz=0.0                          0.089                          0.0 rpy=-1.570796327                         0.0                         0.0 -> xyz=0.0                          0.073                          -0.0763 rpy=-1.570796327                         0.0                         0.0

File: indy_description/urdf_files/opti5.urdf (robot description, URDF)
Before this commit: robot indy, 9 links, 8 joints
Links:
- link link0: mass 13.983 -> 8.329997
- link link1: mass 10.239 -> 8.056963
- link link2: mass 12.857 -> 4.250191
- link link3: mass 7.462 -> 2.816594
- link link4: mass 4.38 -> 4.500514
- link link5: mass 1.656 -> 2.764657
- link link6: mass 0.272 -> 0.377571
Joints:
- joint joint0: limit lower=-2.9670597283903604 upper=2.9670597283903604 effort=431.97 velocity=6.632251157578453 -> lower=-3.141592653589793 upper=3.141592653589793 effort=431.97 velocity=2.775073510670984; origin xyz=0.0                          0.0                          0.19825 rpy=0.0                         0.0                         0.0 -> xyz=0.0                          0.0                          0.257 rpy=0.0                         0.0                         0.0
- joint joint1: limit lower=-1.7453292519943295 upper=2.356194490192345 effort=431.97 velocity=5.585053606381854 -> lower=-3.141592653589793 upper=3.141592653589793 effort=431.97 velocity=2.775073510670984; origin xyz=0.025                          0.0                          0.202 rpy=-1.570796327                         0.0                         0.0 -> xyz=0.0                          -0.0845                          0.084 rpy=1.570796327                         0.0                         0.0
- joint joint2: limit lower=-2.0943951023931953 upper=2.722713633111154 effort=197.23 velocity=6.806784082777885 -> lower=-3.141592653589793 upper=3.141592653589793 effort=209.33 velocity=2.775073510670984; origin xyz=0.0                          -0.463                          0.0 rpy=0.0                         0.0                         0.0 -> xyz=0.0                          0.45                          -0.0005 rpy=0.0                         0.0                         0.0
- joint joint3: limit lower=-3.490658503988659 upper=3.490658503988659 effort=79.79 velocity=8.552113334772216 -> lower=-3.141592653589793 upper=3.141592653589793 effort=124.23 velocity=3.2986722862692828; origin xyz=-0.035                          -0.182                          0.0 rpy=1.570796327                         1.570796327                         0.0 -> xyz=0.0                          0.055                          -0.0845 rpy=-1.570796327                         0.0                         0.0
- joint joint4: limit lower=-2.356194490192345 upper=2.356194490192345 effort=79.79 velocity=9.861110273767961 -> lower=-3.141592653589793 upper=3.141592653589793 effort=124.23 velocity=3.2986722862692828; origin xyz=0.0                          0.0                          0.25 rpy=1.570796327                         0.0                         -1.570796327 -> xyz=0.0                          0.05                          0.395 rpy=1.570796327                         0.0                         0.0
- joint joint5: limit lower=-6.283185307179586 upper=6.283185307179586 effort=79.79 velocity=14.224433403753785 -> lower=-3.141592653589793 upper=3.141592653589793 effort=124.23 velocity=3.2986722862692828; origin xyz=0.0                          0.089                          0.0 rpy=-1.570796327                         0.0                         0.0 -> xyz=0.0                          0.05                          0.0495 rpy=-1.570796327                         0.0                         0.0
